Commit message: Integrated and tested Mapping

File: urdf/mark_four.urdf (robot description, URDF)
Before this commit: robot mark_four, 7 links, 6 joints
Joints:
- joint base_link_to_kinect_link: origin xyz=-0.12 0 0.06 rpy=0 0 0 -> xyz=-0.12 0 0.06 rpy=0 0 3.14159

Commit message: Added collision and inertial tags to urdf

File: urdf/mark_four.urdf (robot description, URDF)
Before this commit: robot mark_four, 7 links, 6 joints
Links:
- link base_link: mass None -> 0.5; geometry collision box size=0.22 0.20 0.05; visual box size=0.22 0.20 0.05
- link left_wheel: mass None -> 0.1; geometry collision cylinder length=0.01 radius=0.035; visual cylinder length=0.01 radius=0.035
- link right_wheel: mass None -> 0.1; geometry collision cylinder length=0.01 radius=0.035; visual cylinder length=0.01 radius=0.035

Commit message: Reimplemented Wheel's inv kinematic equation for lin velocity

File: urdf/mark_four.urdf (robot description, URDF)
Before this commit: robot mark_four, 7 links, 6 joints
Links:
- link base_link: mass 0.5 -> None
